Commit message: Build working Gazebo differential drive simulation

File: ros2_ws/src/robot_core/description/robot.urdf (robot description, URDF)
Before this commit: robot autonomous_search_robot, 3 links, 2 joints
Links:
- link base_link: mass None -> 5.0
- link left_wheel: mass None -> 0.5
- link right_wheel: mass None -> 0.5
Joints:
- joint left_wheel_joint: axis (none) -> 0 1 0; type fixed -> continuous
- joint right_wheel_joint: axis (none) -> 0 1 0; type fixed -> continuous
